Commit message: add compute maximal_wheel_steering_angle in ros2 control xacro file
Signed-off-by: jean.laneurit <jean.laneurit@inrae.fr>

File: hunter_description/ros2_control/hunter.ros2_control.xacro (robot description, xacro)
@@ -2,5 +2,6 @@
 <robot name="hunter_ros2_control" xmlns:xacro="http://www.ros.org/wiki/xacro">
   <xacro:macro name="hunter_ros2_control" params="mode prefix base_name">
-    <xacro:include filename="$(find romea_mobile_base_description)/ros2_control/base1FAS2RWD.ros2_control.xacro" />
+    <xacro:include
+      filename="$(find romea_mobile_base_description)/ros2_control/base1FAS2RWD.ros2_control.xacro" />
     <xacro:property name="conf" value="$(find hunter_description)/config/hunter.yaml" />
     <xacro:property name="props" value="${load_yaml(conf)}" />
@@ -40,4 +41,6 @@
     <xacro:property name="maximal_axle_steering_angle"
       value="${props['front_axle_steering_control']['command']['maximal_angle']}" />
+    <xacro:property name="maximal_wheel_steering_angle"
+      value="${atan(tan(maximal_axle_steering_angle)/(1-tan(maximal_axle_steering_angle)*front_track/(2*wheelbase)))}" />
     <xacro:property name="maximal_wheel_speed"
       value="${props['rear_wheels_speed_control']['command']['maximal_speed']}" />
