Commit message: add import chassis mesh from github
Signed-off-by: jean.laneurit <jean.laneurit@inrae.fr>

File: hunter_description/urdf/hunter.xacro (robot description, xacro)
@@ -118,16 +118,25 @@
       <xacro:property name="front_wheel_steering_link_y" value="${front_hub_carrier_offset}" />
       <xacro:property name="front_wheel_steering_link_xz" value="0.1" />
+      <!-- <origin xyz="${-body_reference_x} 0 ${chassis_height}" rpy="0 0 ${M_PI/2.0}" />
+        <geometry>
+          <mesh filename="package://adap2e_description/meshes/framev3_05.dae" />
+        </geometry>
+        <material name="grey">
+          <color rgba="0.6 0.6 0.6 1" />
+        </material> -->
       <xacro:chassis>
          <!-- visual chassis -->
          <visual>
             <origin
-               xyz="${aabb_center_x-body_reference_x} ${aabb_center_y}  ${aabb_center_z-chassis_height}"
+               xyz="${aabb_center_x-body_reference_x-0.05} ${aabb_center_y}  ${aabb_center_z-chassis_height+0.1255}"
                rpy="0 0 0" />
             <geometry>
-               <box size="${aabb_length} ${aabb_width} ${aabb_height}" />
+               <mesh filename="package://hunter_description/meshes/chassis.STL" />
+               <!-- <box size="${aabb_length} ${aabb_width} ${aabb_height}" /> -->
             </geometry>
          </visual>
          <!-- visual front steering -->
-         <box size="${front_wheel_steering_link_xz} ${front_wheel_steering_link_y} ${front_wheel_steering_link_xz}" />
+         <box
+            size="${front_wheel_steering_link_xz} ${front_wheel_steering_link_y} ${front_wheel_steering_link_xz}" />
          <!-- visual front wheel -->
          <cylinder length="${front_wheel_width}" radius="${front_wheel_radius}" />

Commit message: description: change way to add visuals in xacro file
Signed-off-by: jean.laneurit <jean.laneurit@inrae.fr>

File: hunter_description/urdf/hunter.xacro (robot description, xacro)
@@ -3,4 +3,7 @@
    <xacro:macro name="hunter" params="mode prefix">
       <xacro:include filename="$(find romea_mobile_base_description)/urdf/base1FASxxx.chassis.xacro" />
+      <xacro:include filename="$(find hunter_description)/urdf/visual/chassis.xacro" />
+      <xacro:include filename="$(find hunter_description)/urdf/visual/wheels.xacro" />
+      <xacro:include filename="$(find hunter_description)/urdf/visual/arms.xacro" />
       <xacro:property name="conf" value="$(find hunter_description)/config/hunter.yaml" />
       <xacro:property name="props" value="${load_yaml(conf)}" />
@@ -83,4 +86,5 @@
          value="${props['control_point'][0]}" />
       <!-- Wheel Properties -->
+      <xacro:property name="front_wheel_x_offset" value="0" />
       <xacro:property name="front_hub_carrier_offset"
          value="${props['geometry']['front_axle']['wheels']['hub_carrier_offset']}" />
@@ -118,29 +122,12 @@
       <xacro:property name="front_wheel_steering_link_y" value="${front_hub_carrier_offset}" />
       <xacro:property name="front_wheel_steering_link_xz" value="0.1" />
-      <!-- <origin xyz="${-body_reference_x} 0 ${chassis_height}" rpy="0 0 ${M_PI/2.0}" />
-        <geometry>
-          <mesh filename="package://adap2e_description/meshes/framev3_05.dae" />
-        </geometry>
-        <material name="grey">
-          <color rgba="0.6 0.6 0.6 1" />
-        </material> -->
       <xacro:chassis>
-         <!-- visual chassis -->
-         <visual>
-            <origin
-               xyz="${aabb_center_x-body_reference_x-0.05} ${aabb_center_y}  ${aabb_center_z-chassis_height+0.1255}"
-               rpy="0 0 0" />
-            <geometry>
-               <mesh filename="package://hunter_description/meshes/chassis.STL" />
-               <!-- <box size="${aabb_length} ${aabb_width} ${aabb_height}" /> -->
-            </geometry>
-         </visual>
-         <!-- visual front steering -->
-         <box
-            size="${front_wheel_steering_link_xz} ${front_wheel_steering_link_y} ${front_wheel_steering_link_xz}" />
-         <!-- visual front wheel -->
-         <cylinder length="${front_wheel_width}" radius="${front_wheel_radius}" />
-         <!-- visual rear wheel -->
-         <cylinder length="${rear_wheel_width}" radius="${rear_wheel_radius}" />
+         <xacro:chassis_visual />
+         <xacro:front_left_arm_visual />
+         <xacro:front_right_arm_visual />
+         <xacro:front_left_wheel_visual />
+         <xacro:front_right_wheel_visual />
+         <xacro:rear_left_wheel_visual />
+         <xacro:rear_right_wheel_visual />
       </xacro:chassis>
    </xacro:macro>

Commit message: fix steering link mass for simulation

File: hunter_description/urdf/hunter.xacro (robot description, xacro)
@@ -103,7 +103,7 @@
       <xacro:property name="maximal_wheel_speed"
          value="${props['rear_wheels_speed_control']['command']['maximal_speed']}" />
-      <xacro:property name="wheel_mass" value="5" />
-      <xacro:property name="front_wheel_mass" value="5" />
-      <xacro:property name="rear_wheel_mass" value="5" />
+      <xacro:property name="wheel_mass" value="2" />
+      <xacro:property name="front_wheel_mass" value="2" />
+      <xacro:property name="rear_wheel_mass" value="2" />
       <!-- Steering Properties -->
       <xacro:property name="maximal_axle_steering_angle"
@@ -119,5 +119,5 @@
       <xacro:property name="front_axle_steering_link_y" value="0.05" />
       <xacro:property name="front_axle_steering_link_z" value="0.05" />
-      <xacro:property name="front_wheel_steering_link_mass" value="1" />
+      <xacro:property name="front_wheel_steering_link_mass" value="5" />
       <xacro:property name="front_wheel_steering_link_y" value="${front_hub_carrier_offset}" />
       <xacro:property name="front_wheel_steering_link_xz" value="0.1" />
